Commit message: perf: add urdf mesh model visualization in rviz, add rviz startup file in empty_world.launch

File: legged_examples/legged_unitree/legged_unitree_description/urdf/common/leg.xacro (robot description, xacro)
@@ -33,5 +33,5 @@
                 </xacro:if>
                 <geometry>
-                    <mesh filename="${mesh_path}/hip.dae"
+                    <mesh filename="package://legged_unitree_description/meshes/$(arg robot_type)/hip.dae"
                           scale="1 1 1"/>
                 </geometry>
@@ -67,9 +67,9 @@
                 <geometry>
                     <xacro:if value="${mirror_dae == True}">
-                        <mesh filename="${mesh_path}/thigh.dae"
+                        <mesh filename="package://legged_unitree_description/meshes/$(arg robot_type)/thigh.dae"
                               scale="1 1 1"/>
                     </xacro:if>
                     <xacro:if value="${mirror_dae == False}">
-                        <mesh filename="${mesh_path}/thigh_mirror.dae"
+                        <mesh filename="package://legged_unitree_description/meshes/$(arg robot_type)/thigh_mirror.dae"
                               scale="1 1 1"/>
                     </xacro:if>
@@ -110,5 +110,5 @@
                 <origin rpy="0 0 0" xyz="0 0 0"/>
                 <geometry>
-                    <mesh filename="${mesh_path}/calf.dae"
+                    <mesh filename="package://legged_unitree_description/meshes/$(arg robot_type)/calf.dae"
                           scale="1 1 1"/>
                 </geometry>

File: legged_examples/legged_unitree/legged_unitree_description/urdf/robot.xacro (robot description, xacro)
@@ -13,5 +13,5 @@
             <origin rpy="0 0 0" xyz="0 0 0"/>
             <geometry>
-                <mesh filename="${mesh_path}/trunk.dae" scale="1 1 1"/>
+                <mesh filename="package://legged_unitree_description/meshes/$(arg robot_type)/trunk.dae" scale="1 1 1"/>
             </geometry>
         </visual>
